File: PCB/KeyFlow Schematic.kicad_sch (KiCad schematic)
At the start: 8 parts, among them SW1 SW_Push, SW2 SW_Push, SW3 SW_Push, SW4 SW_Push, SW5 SW_Push, SW6 SW_Push, SW7 RotaryEncoder, U1 XIAO-RP2040-DIP

Commit message: Clean PCB backups, update schematic, add gitignore
Parts:
- U1: footprint XIAO3:XIAO-RP2040-SMD -> Library:XIAO-RP2040-DIP
Changed lines of the file:
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@@
 			)
 		)
-		(property "Footprint" "XIAO3:XIAO-RP2040-SMD"
+		(property "Footprint" "Library:XIAO-RP2040-DIP"
 			(at 107.188 112.268 0)
 			(effects
